File: GRBL_black_pill_breakout.kicad_pcb (KiCad board)
At the start: 2 copper layers, 100 x 100 mm, 216 parts, among them J1 Screw_Terminal_01x12, J10 Conn_01x01, J11 Conn_01x01, J12 Conn_01x01, J13 Conn_01x01, J14 Conn_01x01, J15 Conn_01x01, J16 Conn_01x01, J17 Conn_01x01, J18 Conn_01x01, J19 Conn_01x01, J2 Screw_Terminal_01x12, J20 Conn_01x01, J21 Conn_01x01, J22 Conn_01x01, J23 Conn_01x01, J24 Conn_01x01, J25 Conn_01x01, J26 Conn_01x01, J27 Conn_01x01, J28 Conn_01x01, J29 Conn_01x01, J3 Screw_Terminal_01x12, J30 Conn_01x01, J31 Conn_01x01, J32 Conn_01x01, J33 Conn_01x01, J34 Conn_01x01, J35 Conn_01x01, J36 Conn_01x01, J37 Conn_01x01, J38 Conn_01x01, J39 Conn_01x01, J4 Screw_Terminal_01x02, J40 Conn_01x01, J41 Conn_01x01, J42 Conn_01x01, J43 Conn_01x01, J44 Conn_01x01, J45 Conn_01x01, J46 Conn_01x01, J47 Conn_01x01, J48 Conn_01x01, J49 Conn_01x01, J5 Screw_Terminal_01x12, J50 Conn_01x01, J51 Conn_01x01, J52 Conn_01x01, J53 Conn_01x01, J54 Conn_01x01, J55 Conn_01x01, J56 Conn_01x01, J57 Conn_01x01, J58 Conn_01x01, J59 Conn_01x01, J6 Screw_Terminal_01x12, J60 Conn_01x01, J61 Conn_01x01, J62 Conn_01x01, J63 Conn_01x01, J64 Conn_01x01, J65 Conn_01x01, J66 Conn_01x01, J67 Conn_01x01, J68 Conn_01x01, J69 Conn_01x01, J7 Screw_Terminal_01x12, J8 Screw_Terminal_01x02, J9 Conn_01x01, Q1 PN2222A, Q10 PN2222A, Q11 PN2222A, Q12 PN2222A, Q13 PN2222A, Q14 PN2222A, Q15 PN2222A, Q16 PN2222A, Q17 PN2222A, Q2 PN2222A, Q3 PN2222A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

Commit message: Flip 12V connectors, update values
Parts:
- J1, J2, J3, J5, J6, J7: footprint GRBL_black_pill_breakout:TerminalBlock_Phoenix_MPT-0,5-12-2.54_1x12_P2.54mm_Horizontal -> TerminalBlock_Phoenix:TerminalBlock_Phoenix_MPT-0,5-12-2.54_1x12_P2.54mm_Horizontal
- J10, J11, J12, J13, J14, J15, J16, J17, J18, J19, J20, J21, J22, J23, J24, J25, J26, J27, J28, J29, J30, J31, J32, J33, J34, J35, J36, J37, J38, J39, J40, J41, J42, J43, J44, J45, J46, J47, J48, J49, J50, J51, J52, J53, J54, J55, J56, J57, J58, J59, J60, J61, J62, J63, J64, J65, J66, J67, J68, J69, J9: footprint GRBL_black_pill_breakout:PinHeader_1x01_P2.54mm_Vertical -> Connector_PinHeader_2.54mm:PinHeader_1x01_P2.54mm_Vertical
- R14, R15, R16, R17, R18, R31, R33, R35, R37, R39, R41, R43, R45, R49, R51, R53, R65: value R -> 1k
- R66, R67: value R -> 3k3
- moved J4 5.12 mm to (127.0, 127.6), turned to 0 degrees
- moved J8 5.06 mm to (192.8, 127.6), turned to 0 degrees
Connections:
- J4 pad 1: GNDD -> +12V
- J4 pad 2: +12V -> GNDD
- J8 pad 1: +12P -> GND
- J8 pad 2: GND -> +12P

Commit message: Update the board according to the official GrblHAL pinout for black pill
Parts:
- R1, R32, R34, R36, R38, R40, R42, R44, R46, R48, R50, R52: value R -> 180
- R10, R11, R12, R13, R2, R3, R4, R5, R6, R7, R8, R9: value R -> 510
- R19, R20, R21, R22, R23, R24, R25, R26, R27, R28, R29, R30, R47, R54, R55, R56, R57, R58, R59, R60, R61, R62, R63, R64: value R -> 1k
- moved J8 0.64 mm to (192.7, 127.0)
- moved J4 0.64 mm to (127.0, 127.0)
Connections:
- J10 pad 1: Net-(J10-Pad1) -> /Y_LIMIT
- J11 pad 1: Net-(J11-Pad1) -> /Z_LIMIT
- J12 pad 1: Net-(J12-Pad1) -> /PROBE
- J13 pad 1: Net-(J13-Pad1) -> /SP_PWM
- J22 pad 1: Net-(J22-Pad1) -> /RESET
- J23 pad 1: Net-(J23-Pad1) -> /FEED_HOLD
- J24 pad 1: Net-(J24-Pad1) -> /CYCLE_START
- J25 pad 1: Net-(J25-Pad1) -> /AUXIN0
- J28 pad 1: Net-(J28-Pad1) -> /SP_EN
- J29 pad 1: Net-(J29-Pad1) -> /STEP_EN
- J30 pad 1: Net-(J30-Pad1) -> /AUXOUT0
- J31 pad 1: Net-(J31-Pad1) -> /AUXOUT1
- J32 pad 1: Net-(J32-Pad1) -> /Z_DIR
- J33 pad 1: Net-(J33-Pad1) -> /Z_STEP
- J34 pad 1: Net-(J34-Pad1) -> /Y_DIR
- J35 pad 1: Net-(J35-Pad1) -> /Y_STEP
- J36 pad 1: Net-(J36-Pad1) -> /X_DIR
- J37 pad 1: Net-(J37-Pad1) -> /X_STEP
- J41 pad 1: /IN1 -> /X_LIMIT
- J42 pad 1: /IN2 -> /Y_LIMIT
- J43 pad 1: /IN3 -> /Z_LIMIT
- J44 pad 1: /IN4 -> /PROBE
- J45 pad 1: /IN5 -> /RESET
- J46 pad 1: /IN6 -> /FEED_HOLD
- J47 pad 1: /IN7 -> /CYCLE_START
- J48 pad 1: /IN8 -> /AUXIN0
- J53 pad 1: Net-(J53-Pad1) -> /X_STEP
- J54 pad 1: Net-(J54-Pad1) -> /X_DIR
- J55 pad 1: Net-(J55-Pad1) -> /Y_STEP
- J56 pad 1: Net-(J56-Pad1) -> /Y_DIR
- J57 pad 1: Net-(J57-Pad1) -> /Z_STEP
- J58 pad 1: Net-(J58-Pad1) -> /Z_DIR
- J59 pad 1: Net-(J59-Pad1) -> /STEP_EN
- J60 pad 1: Net-(J60-Pad1) -> /SP_EN
- J61 pad 1: Net-(J61-Pad1) -> /SP_PWM
- J62 pad 1: Net-(J62-Pad1) -> /AUXOUT0
- J63 pad 1: Net-(J63-Pad1) -> /AUXOUT1
- J9 pad 1: Net-(J9-Pad1) -> /X_LIMIT
- R1 pad 1: /IN1 -> /X_LIMIT
- R14 pad 2: Net-(J53-Pad1) -> /X_STEP
- R15 pad 2: Net-(J54-Pad1) -> /X_DIR
- R16 pad 2: Net-(J55-Pad1) -> /Y_STEP
- R17 pad 2: Net-(J56-Pad1) -> /Y_DIR
- R18 pad 2: Net-(J57-Pad1) -> /Z_STEP
- R31 pad 2: Net-(J58-Pad1) -> /Z_DIR
- R32 pad 1: /IN2 -> /Y_LIMIT
- R33 pad 2: Net-(J59-Pad1) -> /STEP_EN
- R34 pad 1: /IN3 -> /Z_LIMIT
- R35 pad 2: Net-(J60-Pad1) -> /SP_EN
- R36 pad 1: /IN4 -> /PROBE
- R37 pad 2: Net-(J61-Pad1) -> /SP_PWM
- R38 pad 1: /IN5 -> /RESET
- R39 pad 2: Net-(J62-Pad1) -> /AUXOUT0
- R40 pad 1: /IN6 -> /FEED_HOLD
- R41 pad 2: Net-(J63-Pad1) -> /AUXOUT1
- R42 pad 1: /IN7 -> /CYCLE_START
- R44 pad 1: /IN8 -> /AUXIN0
- R47 pad 1: /IN1 -> /X_LIMIT
- R54 pad 1: /IN2 -> /Y_LIMIT
- R55 pad 1: /IN3 -> /Z_LIMIT
- R56 pad 1: /IN4 -> /PROBE
- R57 pad 1: /IN5 -> /RESET
- R58 pad 1: /IN6 -> /FEED_HOLD
- R59 pad 1: /IN7 -> /CYCLE_START
- R60 pad 1: /IN8 -> /AUXIN0
- U1 pad 1: Net-(U1-Pad1) -> unconnected-(U1-Pad1)
- U1 pad 10: Net-(J33-Pad1) -> /Z_STEP
- U1 pad 11: Net-(J32-Pad1) -> /Z_DIR
- U1 pad 12: Net-(J31-Pad1) -> /AUXOUT1
- U1 pad 13: Net-(J30-Pad1) -> /AUXOUT0
- U1 pad 14: Net-(J29-Pad1) -> /STEP_EN
- U1 pad 15: Net-(J28-Pad1) -> /SP_EN
- U1 pad 18: Net-(U1-Pad18) -> unconnected-(U1-Pad18)
- U1 pad 21: Net-(J9-Pad1) -> /X_LIMIT
- U1 pad 22: Net-(J10-Pad1) -> /Y_LIMIT
- U1 pad 23: Net-(J11-Pad1) -> /Z_LIMIT
- U1 pad 24: Net-(J12-Pad1) -> /PROBE
- U1 pad 25: Net-(J13-Pad1) -> /SP_PWM
- U1 pad 34: Net-(J22-Pad1) -> /RESET
- U1 pad 35: Net-(J23-Pad1) -> /FEED_HOLD
- U1 pad 36: Net-(J24-Pad1) -> /CYCLE_START
- U1 pad 37: Net-(J25-Pad1) -> /AUXIN0
- U1 pad 40: Net-(U1-Pad40) -> unconnected-(U1-Pad40)
- U1 pad 5: Net-(U1-Pad5) -> unconnected-(U1-Pad5)
- U1 pad 6: Net-(J37-Pad1) -> /X_STEP
- U1 pad 7: Net-(J36-Pad1) -> /X_DIR
- U1 pad 8: Net-(J35-Pad1) -> /Y_STEP
- U1 pad 9: Net-(J34-Pad1) -> /Y_DIR
Routing:
- net /SP_PWM: track 0.00 -> 87.5 mm, vias 0 -> 2
- net /X_STEP: track 0.00 -> 53.4 mm, vias 0 -> 2
- net /SP_EN: track 0.00 -> 50.4 mm, vias 0 -> 1
- net /AUXOUT1: track 0.00 -> 49.1 mm, vias 0 -> 2
- net /AUXOUT0: track 0.00 -> 48.6 mm, vias 0 -> 2
- net /STEP_EN: track 0.00 -> 47.2 mm, vias 0 -> 1
- net /X_DIR: track 0.00 -> 45.7 mm, vias 0 -> 2
- net /Y_STEP: track 0.00 -> 38.7 mm, vias 0 -> 2
- net /Z_DIR: track 0.00 -> 38.2 mm, vias 0 -> 2
- net /Z_STEP: track 0.00 -> 35.4 mm, vias 0 -> 2
- net /Y_DIR: track 0.00 -> 32.0 mm
- net Net-(J53-Pad1): track 25.1 -> 0.00 mm
- net /PROBE: track 0.00 -> 23.1 mm
- net Net-(J54-Pad1): track 22.6 -> 0.00 mm
- net /Z_LIMIT: track 0.00 -> 20.9 mm
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Other:
- net class Default removed
